Commit message: Integrate Gen 2.1 controls, preserve version history, and add Gen 2 trial photos

File: shared/simulation/pybullet/snake.urdf (robot description, URDF)
Before this commit: robot snake, 10 links, 9 joints
Links:
- added link link10, mass 0.1; collision box size=0.058 0.055 0.055; visual box size=0.058 0.055 0.055
- link link0: geometry collision box size=0.058 0.055 0.055; visual box size=0.058 0.055 0.055
- link link1: geometry collision box size=0.058 0.055 0.055; visual box size=0.058 0.055 0.055
- link link2: geometry collision box size=0.058 0.055 0.055; visual box size=0.058 0.055 0.055
- link link3: geometry collision box size=0.058 0.055 0.055; visual box size=0.058 0.055 0.055
- link link4: geometry collision box size=0.058 0.055 0.055; visual box size=0.058 0.055 0.055
- link link5: geometry collision box size=0.058 0.055 0.055; visual box size=0.058 0.055 0.055
- link link6: geometry collision box size=0.058 0.055 0.055; visual box size=0.058 0.055 0.055
- link link7: geometry collision box size=0.058 0.055 0.055; visual box size=0.058 0.055 0.055
- link link8: geometry collision box size=0.058 0.055 0.055; visual box size=0.058 0.055 0.055
- link link9: geometry collision box size=0.058 0.055 0.055; visual box size=0.058 0.055 0.055
Joints:
- added joint joint9: type revolute, parent link9, child link10, origin xyz=0.058 0 0, axis 0 0 1, limit lower=-1.22173 upper=1.22173 effort=10 velocity=5
- joint joint0: limit lower=-1.5 upper=1.5 effort=10 velocity=5 -> lower=-1.22173 upper=1.22173 effort=10 velocity=5; origin xyz=0.06 0 0 -> xyz=0.058 0 0
- joint joint1: limit lower=-1.5 upper=1.5 effort=10 velocity=5 -> lower=-1.22173 upper=1.22173 effort=10 velocity=5; origin xyz=0.06 0 0 -> xyz=0.058 0 0
- joint joint2: limit lower=-1.5 upper=1.5 effort=10 velocity=5 -> lower=-1.22173 upper=1.22173 effort=10 velocity=5; origin xyz=0.06 0 0 -> xyz=0.058 0 0
- joint joint3: limit lower=-1.5 upper=1.5 effort=10 velocity=5 -> lower=-1.22173 upper=1.22173 effort=10 velocity=5; origin xyz=0.06 0 0 -> xyz=0.058 0 0
- joint joint4: limit lower=-1.5 upper=1.5 effort=10 velocity=5 -> lower=-1.22173 upper=1.22173 effort=10 velocity=5; origin xyz=0.06 0 0 -> xyz=0.058 0 0
- joint joint5: limit lower=-1.5 upper=1.5 effort=10 velocity=5 -> lower=-1.22173 upper=1.22173 effort=10 velocity=5; origin xyz=0.06 0 0 -> xyz=0.058 0 0
- joint joint6: limit lower=-1.5 upper=1.5 effort=10 velocity=5 -> lower=-1.22173 upper=1.22173 effort=10 velocity=5; origin xyz=0.06 0 0 -> xyz=0.058 0 0
- joint joint7: limit lower=-1.5 upper=1.5 effort=10 velocity=5 -> lower=-1.22173 upper=1.22173 effort=10 velocity=5; origin xyz=0.06 0 0 -> xyz=0.058 0 0
- joint joint8: limit lower=-1.5 upper=1.5 effort=10 velocity=5 -> lower=-1.22173 upper=1.22173 effort=10 velocity=5; origin xyz=0.06 0 0 -> xyz=0.058 0 0
